File: breakout.kicad_pcb (KiCad board)
At the start: 2 copper layers, 5 parts, among them P1 CONN_12, P2 CONN_12, P3 CONN_12, P4 CONN_12, U1 MK20LF

Commit message: almost finished v1
Parts:
- added C1: CP1, SM0805, F.Cu at (102.0, 105.3)
- added C2: C, SM0805, F.Cu at (108.6, 105.3)
- added C3: C, SM0805, F.Cu at (136.0, 100.5)
- added C4: CP1, SM0805, F.Cu at (132.9, 93.7)
- added C5: C, SM0805, F.Cu at (138.6, 101.9)
- added C6: C, SM0805, F.Cu at (137.0, 111.1)
- added C7: C, SM0805, F.Cu at (151.9, 114.2)
- added C8: C, SM0805, B.Cu at (169.4, 118.1)
- added K1: CONN_3, SIL-3, F.Cu at (129.4, 96.4)
- added K2: CONN_3, SIL-3, F.Cu at (137.0, 121.0)
- added P5: CONN_12, SIL-12, F.Cu at (149.5, 87.8)
- added P6: CONN_5, SIL-5, F.Cu at (147.3, 121.1)
- added P7: CONN_1, SIL-1, F.Cu at (163.3, 121.0)
- added R1: R, SM0805, F.Cu at (124.9, 101.9)
- added R2: R, SM0805, F.Cu at (125.0, 104.6)
- added RESET2: CONN_1, 1pin, F.Cu at (101.1, 120.0)
- added RIGHT1: CONN_12, SIL-12, F.Cu at (166.1, 104.3)
- P1, P3, P4: value CONN_12 -> CONN_2; footprint SIL-12 -> SIL-2
- P2: value CONN_12 -> CONN_4; footprint SIL-12 -> SIL-4
- moved P2 37.3 mm to (114.6, 105.3), turned to 90 degrees
- moved P4 36.0 mm to (129.6, 111.4), turned to 90 degrees
- moved P3 25.2 mm to (129.7, 103.2), turned to 90 degrees
- moved P1 16.2 mm to (129.3, 89.0), turned to 270 degrees
Connections:
- P1 pad 1: N-0000047 -> N-0000015
- P1 pad 2: N-0000046 -> N-000005
- P2 pad 1: N-000006 -> N-0000015
- P2 pad 2: N-000007 -> N-0000014
- P2 pad 3: N-000008 -> N-0000013
- P2 pad 4: N-000009 -> N-0000045
- P3 pad 1: N-0000029 -> N-0000044
- P3 pad 2: N-0000030 -> N-0000043
- P4 pad 1: N-0000018 -> N-000009
- P4 pad 2: N-0000048 -> N-0000012
- U1 pad 1: N-0000037 -> N-0000010
- U1 pad 10: N-0000045 -> N-0000010
- U1 pad 11: N-0000046 -> N-0000015
- U1 pad 12: N-0000047 -> N-0000015
- U1 pad 13: N-000005 -> N-0000041
- U1 pad 14: N-000004 -> N-0000040
- U1 pad 15: N-000003 -> N-0000039
- U1 pad 16: N-000002 -> N-0000010
- U1 pad 17: N-0000011 -> N-0000025
- U1 pad 18: N-0000035 -> N-0000032
- U1 pad 19: N-0000034 -> N-0000036
- U1 pad 2: N-0000038 -> N-0000015
- U1 pad 20: N-0000033 -> N-0000017
- U1 pad 21: N-0000032 -> N-0000016
- U1 pad 22: N-0000031 -> N-0000010
- U1 pad 23: N-0000030 -> N-0000015
- U1 pad 24: N-0000029 -> N-0000042
- U1 pad 25: N-0000028 -> N-0000024
- U1 pad 26: N-0000019 -> N-0000021
- U1 pad 27: N-0000027 -> N-0000029
- U1 pad 28: N-0000026 -> N-0000033
- U1 pad 29: N-0000025 -> N-0000037
- U1 pad 3: N-0000039 -> N-0000043
- U1 pad 30: N-0000024 -> N-000002
- U1 pad 31: N-0000023 -> N-000004
- U1 pad 32: N-0000022 -> N-000003
- U1 pad 33: N-0000021 -> N-0000028
- U1 pad 34: N-0000020 -> N-0000026
- U1 pad 35: N-0000048 -> N-0000023
- U1 pad 36: N-0000018 -> N-0000020
- U1 pad 37: N-0000017 -> N-0000030
- U1 pad 38: N-0000016 -> N-0000034
- U1 pad 39: N-0000015 -> N-0000038
- U1 pad 4: N-0000040 -> N-0000044
- U1 pad 40: N-0000014 -> N-000008
- U1 pad 41: N-0000013 -> N-000007
- U1 pad 42: N-0000012 -> N-000006
- U1 pad 43: N-000001 -> N-0000027
- U1 pad 44: N-0000010 -> N-0000018
- U1 pad 45: N-000009 -> N-0000022
- U1 pad 46: N-000008 -> N-0000019
- U1 pad 47: N-000007 -> N-0000031
- U1 pad 48: N-000006 -> N-0000035
- U1 pad 5: N-0000036 -> N-0000011
- U1 pad 6: N-0000041 -> N-0000045
- U1 pad 7: N-0000042 -> N-0000012
- U1 pad 8: N-0000043 -> N-000009
- U1 pad 9: N-0000044 -> N-0000010
Routing:
- net N-0000015: track 14.8 -> 235.6 mm
- net (no net): track 90.5 -> 0.00 mm
- net N-0000010: track 12.6 -> 52.4 mm
- net N-0000045: track 16.2 -> 53.1 mm
- net N-0000011: track 0.00 -> 31.7 mm, vias 0 -> 2
- net N-0000021: track 0.00 -> 22.7 mm
- net N-0000030: track 0.00 -> 18.7 mm
- net N-0000020: track 0.00 -> 18.4 mm
- net N-0000024: track 0.00 -> 17.7 mm
- net N-0000023: track 0.00 -> 17.5 mm
- net N-000009: track 0.00 -> 17.4 mm
- net N-0000047: track 17.3 -> 0.00 mm
- net N-0000035: track 0.00 -> 17.2 mm
- net N-0000034: track 0.00 -> 17.2 mm
- net N-0000046: track 17.2 -> 0.00 mm
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Other:
- rule trace_min: 0.254 -> 0.1
- rule via_min_size: 0.889 -> 0.1
