File: breakout.sch (KiCad schematic (older format))
At the start: 48 parts, among them U1 MK20LF

Commit message: almost finished v1
Parts:
- removed DM0, DP0, P? (x28), PTD0, PTD1, PTD2, PTD3, PTD4, PTD5, PTD6, PTD7, USB (x5): CONN_1, symbol CONN_1
- added C1, C4: CP1, symbol CP1
- added C2, C3, C5, C6, C7: C, symbol C
- added K1, K2: CONN_3, symbol CONN_3
- added P1, P3, P4: CONN_2, symbol CONN_2
- added P2: CONN_4, symbol CONN_4
- added P5, RIGHT1: CONN_12, symbol CONN_12
- added P6: CONN_5, symbol CONN_5
- added P7: CONN_1, symbol CONN_1
- gave numbers to parts that had none: 4
Connections:
- wire segments 65 -> 118

Commit message: finished board
Connections:
- wire segments 118 -> 120
Changed lines of the file:
@@
 LIBS:inductor_select
 LIBS:logo
-LIBS:mchck-cache
 LIBS:mcp1702
 LIBS:mcp73831
@@
 LIBS:vdda
 LIBS:vssa
+LIBS:breakout-cache
 EELAYER 24 0
 EELAYER END
@@
 $EndComp
 Connection ~ 6800 4450
+Wire Wire Line
+	7350 4900 6800 4900
+Wire Wire Line
+	6800 4900 6800 4450
 $EndSCHEMATC
